File: Macropad.kicad_sch (KiCad schematic)
At the start: 50 parts, among them SW1 SW_Push, SW10 SW_Push, SW11 SW_Push, SW12 SW_Push, SW2 SW_Push, SW3 SW_Push, SW4 SW_Push, SW5 SW_Push, SW6 SW_Push, SW7 SW_Push, SW8 SW_Push, SW9 SW_Push

Commit message: Final Version
Signed-off-by: Kozova1 <mug66kk@gmail.com>
Parts:
- LED1, LED10, LED11, LED12, LED2, LED3, LED4, LED5, LED6, LED7, LED8, LED9: footprint kicad-keyboard-parts:MX_SK6812MINI-E_REV -> Sk6812ReverseMount:MX_SK6812MINI-E
Changed lines of the file:
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@@
       (effects (font (size 1.27 1.27)) (justify left))
     )
-    (property "Footprint" "kicad-keyboard-parts:MX_SK6812MINI-E_REV" (id 2) (at 63.5 120.65 0)
+    (property "Footprint" "Sk6812ReverseMount:MX_SK6812MINI-E" (id 2) (at 63.5 120.65 0)
       (effects (font (size 1.27 1.27)) (justify left top) hide)
     )
@@
       (effects (font (size 1.27 1.27)) (justify left))
     )
-    (property "Footprint" "kicad-keyboard-parts:MX_SK6812MINI-E_REV" (id 2) (at 63.5 151.13 0)
+    (property "Footprint" "Sk6812ReverseMount:MX_SK6812MINI-E" (id 2) (at 63.5 151.13 0)
       (effects (font (size 1.27 1.27)) (justify left top) hide)
     )
@@
       (effects (font (size 1.27 1.27)) (justify left))
     )
-    (property "Footprint" "kicad-keyboard-parts:MX_SK6812MINI-E_REV" (id 2) (at 63.5 181.61 0)
+    (property "Footprint" "Sk6812ReverseMount:MX_SK6812MINI-E" (id 2) (at 63.5 181.61 0)
       (effects (font (size 1.27 1.27)) (justify left top) hide)
     )
@@
       (effects (font (size 1.27 1.27)) (justify left))
     )
-    (property "Footprint" "kicad-keyboard-parts:MX_SK6812MINI-E_REV" (id 2) (at 88.9 120.65 0)
+    (property "Footprint" "Sk6812ReverseMount:MX_SK6812MINI-E" (id 2) (at 88.9 120.65 0)
       (effects (font (size 1.27 1.27)) (justify left top) hide)
     )
@@
       (effects (font (size 1.27 1.27)) (justify left))
     )
-    (property "Footprint" "kicad-keyboard-parts:MX_SK6812MINI-E_REV" (id 2) (at 88.9 151.13 0)
+    (property "Footprint" "Sk6812ReverseMount:MX_SK6812MINI-E" (id 2) (at 88.9 151.13 0)
       (effects (font (size 1.27 1.27)) (justify left top) hide)
     )
@@
       (effects (font (size 1.27 1.27)) (justify left))
     )
-    (property "Footprint" "kicad-keyboard-parts:MX_SK6812MINI-E_REV" (id 2) (at 88.9 181.61 0)
+    (property "Footprint" "Sk6812ReverseMount:MX_SK6812MINI-E" (id 2) (at 88.9 181.61 0)
       (effects (font (size 1.27 1.27)) (justify left top) hide)
     )
@@
       (effects (font (size 1.27 1.27)) (justify left))
     )
-    (property "Footprint" "kicad-keyboard-parts:MX_SK6812MINI-E_REV" (id 2) (at 114.3 120.65 0)
+    (property "Footprint" "Sk6812ReverseMount:MX_SK6812MINI-E" (id 2) (at 114.3 120.65 0)
       (effects (font (size 1.27 1.27)) (justify left top) hide)
     )
@@
       (effects (font (size 1.27 1.27)) (justify left))
     )
-    (property "Footprint" "kicad-keyboard-parts:MX_SK6812MINI-E_REV" (id 2) (at 114.3 151.13 0)
+    (property "Footprint" "Sk6812ReverseMount:MX_SK6812MINI-E" (id 2) (at 114.3 151.13 0)
       (effects (font (size 1.27 1.27)) (justify left top) hide)
     )
@@
       (effects (font (size 1.27 1.27)) (justify left))
     )
-    (property "Footprint" "kicad-keyboard-parts:MX_SK6812MINI-E_REV" (id 2) (at 114.3 181.61 0)
+    (property "Footprint" "Sk6812ReverseMount:MX_SK6812MINI-E" (id 2) (at 114.3 181.61 0)
       (effects (font (size 1.27 1.27)) (justify left top) hide)
     )
@@
       (effects (font (size 1.27 1.27)) (justify left))
     )
-    (property "Footprint" "kicad-keyboard-parts:MX_SK6812MINI-E_REV" (id 2) (at 139.7 120.65 0)
+    (property "Footprint" "Sk6812ReverseMount:MX_SK6812MINI-E" (id 2) (at 139.7 120.65 0)
       (effects (font (size 1.27 1.27)) (justify left top) hide)
     )
@@
       (effects (font (size 1.27 1.27)) (justify left))
     )
-    (property "Footprint" "kicad-keyboard-parts:MX_SK6812MINI-E_REV" (id 2) (at 139.7 151.13 0)
+    (property "Footprint" "Sk6812ReverseMount:MX_SK6812MINI-E" (id 2) (at 139.7 151.13 0)
       (effects (font (size 1.27 1.27)) (justify left top) hide)
     )
@@
       (effects (font (size 1.27 1.27)) (justify left))
     )
-    (property "Footprint" "kicad-keyboard-parts:MX_SK6812MINI-E_REV" (id 2) (at 139.7 181.61 0)
+    (property "Footprint" "Sk6812ReverseMount:MX_SK6812MINI-E" (id 2) (at 139.7 181.61 0)
       (effects (font (size 1.27 1.27)) (justify left top) hide)
     )
@@
     )
     (path "/00000000-0000-0000-0000-0000612112f5"
-      (reference "LED1") (unit 1) (value "SK6812") (footprint "kicad-keyboard-parts:MX_SK6812MINI-E_REV")
+      (reference "LED1") (unit 1) (value "SK6812") (footprint "Sk6812ReverseMount:MX_SK6812MINI-E")
     )
     (path "/00000000-0000-0000-0000-000061229b69"
-      (reference "LED2") (unit 1) (value "SK6812") (footprint "kicad-keyboard-parts:MX_SK6812MINI-E_REV")
+      (reference "LED2") (unit 1) (value "SK6812") (footprint "Sk6812ReverseMount:MX_SK6812MINI-E")
     )
     (path "/00000000-0000-0000-0000-00006122f939"
-      (reference "LED3") (unit 1) (value "SK6812") (footprint "kicad-keyboard-parts:MX_SK6812MINI-E_REV")
+      (reference "LED3") (unit 1) (value "SK6812") (footprint "Sk6812ReverseMount:MX_SK6812MINI-E")
     )
     (path "/00000000-0000-0000-0000-00006122f959"
-      (reference "LED4") (unit 1) (value "SK6812") (footprint "kicad-keyboard-parts:MX_SK6812MINI-E_REV")
+      (reference "LED4") (unit 1) (value "SK6812") (footprint "Sk6812ReverseMount:MX_SK6812MINI-E")
     )
     (path "/00000000-0000-0000-0000-00006129524c"
-      (reference "LED5") (unit 1) (value "SK6812") (footprint "kicad-keyboard-parts:MX_SK6812MINI-E_REV")
+      (reference "LED5") (unit 1) (value "SK6812") (footprint "Sk6812ReverseMount:MX_SK6812MINI-E")
     )
     (path "/00000000-0000-0000-0000-00006129526c"
-      (reference "LED6") (unit 1) (value "SK6812") (footprint "kicad-keyboard-parts:MX_SK6812MINI-E_REV")
+      (reference "LED6") (unit 1) (value "SK6812") (footprint "Sk6812ReverseMount:MX_SK6812MINI-E")
     )
     (path "/00000000-0000-0000-0000-00006129528c"
-      (reference "LED7") (unit 1) (value "SK6812") (footprint "kicad-keyboard-parts:MX_SK6812MINI-E_REV")
+      (reference "LED7") (unit 1) (value "SK6812") (footprint "Sk6812ReverseMount:MX_SK6812MINI-E")
     )
     (path "/00000000-0000-0000-0000-0000612952ac"
-      (reference "LED8") (unit 1) (value "SK6812") (footprint "kicad-keyboard-parts:MX_SK6812MINI-E_REV")
+      (reference "LED8") (unit 1) (value "SK6812") (footprint "Sk6812ReverseMount:MX_SK6812MINI-E")
     )
     (path "/00000000-0000-0000-0000-0000612af78e"
-      (reference "LED9") (unit 1) (value "SK6812") (footprint "kicad-keyboard-parts:MX_SK6812MINI-E_REV")
+      (reference "LED9") (unit 1) (value "SK6812") (footprint "Sk6812ReverseMount:MX_SK6812MINI-E")
     )
     (path "/00000000-0000-0000-0000-0000612af7ae"
-      (reference "LED10") (unit 1) (value "SK6812") (footprint "kicad-keyboard-parts:MX_SK6812MINI-E_REV")
+      (reference "LED10") (unit 1) (value "SK6812") (footprint "Sk6812ReverseMount:MX_SK6812MINI-E")
     )
     (path "/00000000-0000-0000-0000-0000612af7ce"
-      (reference "LED11") (unit 1) (value "SK6812") (footprint "kicad-keyboard-parts:MX_SK6812MINI-E_REV")
+      (reference "LED11") (unit 1) (value "SK6812") (footprint "Sk6812ReverseMount:MX_SK6812MINI-E")
     )
     (path "/00000000-0000-0000-0000-0000612af7ee"
-      (reference "LED12") (unit 1) (value "SK6812") (footprint "kicad-keyboard-parts:MX_SK6812MINI-E_REV")
+      (reference "LED12") (unit 1) (value "SK6812") (footprint "Sk6812ReverseMount:MX_SK6812MINI-E")
     )
     (path "/00000000-0000-0000-0000-0000611e5ba6"
